Commit message: Updated Base Model file

File: urdf/Body_Assm.urdf (robot description, URDF)
Before this commit: robot Body_Assm, 4 links, 3 joints
Links:
- link front_wheels: mass 3.8822 -> 3.8893
- link rear_wheels: mass 3.8822 -> 3.8893
Joints:
- joint dummy_joint: origin (none) -> xyz=0 0 0.1 rpy=0 0 0
- joint front_wheel_joint: origin xyz=0.14367 -0.4883 0.54124 rpy=1.5708 0.59058 1.5708 -> xyz=-0.07 -0.1 0.022 rpy=1.5708 0 0
- joint rear_wheel_joint: origin xyz=0.14367 -0.9383 0.54124 rpy=-1.5708 -0.1362 1.5708 -> xyz=-0.52 -0.1 0.022 rpy=1.5708 0 0

File: urdf/rover.urdf.xacro (robot description, xacro)
@@ -6,5 +6,5 @@
   name="body_arm_joint" type="fixed" >
   <origin
-    xyz="0 0 0"
+    xyz="-0.15 0.395 0.063"
     rpy="0 0 0" />
     <parent
