Commit message: Updated rover urdf adding dummy link

File: urdf/Rover.urdf (robot description, URDF)
Before this commit: robot rover, 8 links, 7 joints
Links:
- added link world
Joints:
- added joint dummy_joint: type continuous, parent world, child base_link, origin xyz=0.0 0.0 0.1 rpy=0 0 0, axis 0 0 1

Commit message: Added lidar in urdf

File: urdf/Rover.urdf (robot description, URDF)
Before this commit: robot rover, 9 links, 8 joints
Links:
- added link base_laser, mass 0.15717; collision mesh filename=package://bot/meshes/ydlidar.dae; visual mesh filename=package://bot/meshes/ydlidar.dae
- added link laser_frame, mass 0.25482
Joints:
- added joint hokuyo_joint: type fixed, parent base_link, child base_laser, origin xyz=-0.02 0.3 0.063 rpy=0 0 0, axis 0 1 0
- added joint laser_joint: type fixed, parent base_laser, child laser_frame, origin xyz=0 0 0.03172 rpy=0 0 0, axis 0 0 0

Commit message: Added controllers for base and extended it with the arm controllers.

File: urdf/Rover.urdf (robot description, URDF)
Before this commit: robot rover, 9 links, 8 joints
Links:
- removed link front_wheels
- added link front_left, mass 1.7624; collision mesh filename=package://rover/meshes/front_left.STL; visual mesh filename=package://rover/meshes/front_left.STL
- added link front_right, mass 1.7624; collision mesh filename=package://rover/meshes/front_right.STL; visual mesh filename=package://rover/meshes/front_right.STL
- link base_link: mass 13.103 -> 13.26
Joints:
- removed joint front_wheel_joint
- added joint front_left_joint: type continuous, parent base_link, child front_left, origin xyz=-0.07 0.5 0.01 rpy=1.5708 0 0, axis 0 0 1
- added joint front_right_joint: type continuous, parent base_link, child front_right, origin xyz=-0.07 -0.1 0.01 rpy=1.5708 0 0, axis 0 0 1
- joint dummy_joint: axis 0 0 1 -> (none); type continuous -> fixed
- joint rear_wheel_joint: origin xyz=-0.52 -0.1 0.022 rpy=1.5708 0 0 -> xyz=-0.52 -0.1 0.01 rpy=1.5708 0 0

Commit message: Robot moves

File: urdf/Rover.urdf (robot description, URDF)
Before this commit: robot rover, 12 links, 11 joints
Links:
- removed link world
- added link dummy
- link base_laser: geometry collision mesh filename=package://rover/meshes/ydlidar.dae; visual mesh filename=package://rover/meshes/ydlidar.dae
- link laser_frame: geometry collision mesh filename=package://rover/meshes/ydlidar.dae; visual mesh filename=package://rover/meshes/ydlidar.dae
Joints:
- joint dummy_joint: parent world -> dummy
- joint hokuyo_joint: origin xyz=-0.02 0.3 0.063 rpy=0 0 0 -> xyz=0.08 0.2 0.013 rpy=0 0 0
