Commit message: Added xacro file

File: urdf/Arm.urdf (robot description, URDF)
Before this commit: robot Arm, 5 links, 4 joints
Links:
- link arn_base: geometry collision mesh filename=package://rover/meshes/arn_base.STL; visual mesh filename=package://rover/meshes/arn_base.STL
- link bicep: geometry collision mesh filename=package://rover/meshes/bicep.STL; visual mesh filename=package://rover/meshes/bicep.STL
- link bottom_wrist: geometry collision mesh filename=package://rover/meshes/bottom_wrist.STL; visual mesh filename=package://rover/meshes/bottom_wrist.STL
- link elbow: geometry collision mesh filename=package://rover/meshes/elbow.STL; visual mesh filename=package://rover/meshes/elbow.STL
- link top_wrist: geometry collision mesh filename=package://rover/meshes/top_wrist.STL; visual mesh filename=package://rover/meshes/top_wrist.STL

File: urdf/rover.urdf.xacro (robot description, xacro)
@@ -1,4 +1,15 @@
 <?xml version="1.0"?>
 <robot xmlns:xacro="http://ros.org/wiki/xacro" name="rover" >
-  <xacro:include filename="rover.urdf"/>
+  <xacro:include filename="$(find rover)/urdf/Body_Assm.urdf"/>
+  <xacro:include filename="$(find rover)/urdf/Arm.urdf" />
+  <joint
+  name="body_arm_joint" type="fixed" >
+  <origin
+    xyz="0 0 0"
+    rpy="0 0 0" />
+    <parent
+      link="base_link" />
+    <child
+      link="arn_base" />
+  </joint>
 </robot>

Commit message: Added rover controllers and transmission

File: urdf/Arm.urdf (robot description, URDF)
Before this commit: robot Arm, 5 links, 4 joints
Links:
- added link world
Joints:
- added joint arn_base_joint: type continuous, parent world, child arn_base, origin xyz=0.0 0.0 0.1 rpy=0 0 0, axis 0 0 1

File: urdf/Body_Assm.urdf (robot description, URDF)
Before this commit: robot rover, 4 links, 3 joints
Links:
- removed link world
Joints:
- removed joint dummy_joint

File: urdf/rover.urdf.xacro (robot description, xacro)
@@ -4,5 +4,5 @@
   <xacro:include filename="$(find rover)/urdf/Arm.urdf" />
   <joint
-  name="body_arm_joint" type="fixed" >
+  name="arn_base_joint" type="fixed" >
   <origin
     xyz="-0.15 0.395 0.063"
@@ -13,3 +13,11 @@
       link="arn_base" />
   </joint>
+<!--######################################################################-->
+<gazebo>
+    <plugin name="gazebo_ros_control" filename="libgazebo_ros_control.so">
+      <robotNamespace>/</robotNamespace>
+      <controlPeriod>0.001</controlPeriod>
+      <legacyModeNS>false</legacyModeNS>
+    </plugin>
+</gazebo>
 </robot>

Commit message: No errors. Full xacro integration. Robot is controlled with teleop.

File: urdf/Arm.urdf (robot description, URDF)
Before this commit: robot Arm, 6 links, 5 joints
Links:
- removed link world
Joints:
- removed joint arn_base_joint

File: urdf/Body_Assm.urdf (robot description, URDF)
Before this commit: robot rover, 3 links, 2 joints
Links:
- removed link front_wheels
- added link dummy
- added link front_left, mass 1.7624; collision mesh filename=package://rover/meshes/front_left.STL; visual mesh filename=package://rover/meshes/front_left.STL
- added link front_right, mass 1.7624; collision mesh filename=package://rover/meshes/front_right.STL; visual mesh filename=package://rover/meshes/front_right.STL
- link base_link: mass 13.103 -> 13.26
Joints:
- removed joint front_wheel_joint
- added joint front_left_joint: type continuous, parent base_link, child front_left, origin xyz=-0.07 0.5 0.01 rpy=1.5708 0 0, axis 0 0 1
- added joint front_right_joint: type continuous, parent base_link, child front_right, origin xyz=-0.07 -0.1 0.01 rpy=1.5708 0 0, axis 0 0 1
- joint rear_wheel_joint: origin xyz=-0.52 -0.1 0.022 rpy=1.5708 0 0 -> xyz=-0.52 -0.1 0.01 rpy=1.5708 0 0

File: urdf/rover.urdf.xacro (robot description, xacro)
@@ -3,13 +3,20 @@
   <xacro:include filename="$(find rover)/urdf/Body_Assm.urdf"/>
   <xacro:include filename="$(find rover)/urdf/Arm.urdf" />
-  <joint
-  name="arn_base_joint" type="fixed" >
-  <origin
-    xyz="-0.15 0.395 0.063"
-    rpy="0 0 0" />
-    <parent
-      link="base_link" />
-    <child
-      link="arn_base" />
+  <xacro:include filename="$(find rover)/urdf/ydlidar.urdf" />
+  <joint name="arn_base_joint" type="fixed">
+    <origin rpy="0 0 0" xyz="-0.15 0.395 0.063"/>
+    <parent link="base_link"/>
+    <child link="arn_base"/>
+  </joint>
+  <joint name="dummy_joint" type="fixed">
+    <origin rpy="0 0 0" xyz="0.0 0.0 0.1"/>
+    <parent link="dummy"/>
+    <child link="base_link"/>
+  </joint>
+  <joint type="fixed" name="hokuyo_joint">
+    <origin xyz="0.08 0.2 0.013" rpy="0 0 0"/>
+    <child link="base_laser"/>
+    <parent link="base_link"/>
+    <axis xyz="0 1 0" rpy="0 0 0"/>
   </joint>
 <!--######################################################################-->
