Commit message: Integrated lidar and added laserscan.py script to extract info from lidar

File: urdf/newrover.urdf (robot description, URDF)
Before this commit: robot rover, 11 links, 10 joints
Links:
- link base_laser: geometry collision mesh filename=package://rover/meshes/ydlidar.dae; visual mesh filename=package://rover/meshes/ydlidar.dae
- link laser_frame: geometry collision mesh filename=package://rover/meshes/ydlidar.dae; visual mesh filename=package://rover/meshes/ydlidar.dae

File: urdf/rover.urdf.xacro (robot description, xacro)
@@ -20,8 +20,43 @@
     <axis xyz="0 1 0" rpy="0 0 0"/>
   </joint>
+  <gazebo reference="base_laser">
+		<gravity>true</gravity>
+		<!-- Gazebo has fixed set of Sensors types. Check them out here <> -->
+		<sensor name="laser" type="ray">
+			<!-- Add in your sensor characteristics -->
+			<pose> 0 0 0 0 0 0 </pose>
+			<visualise>true</visualise>
+			<update_rate>40</update_rate>
+			<always_on>true</always_on>
+			<ray>
+				<scan>
+					<horizontal>
+						<samples>720</samples>
+						<resolution>1</resolution>
+						<min_angle>-1.570796</min_angle>
+              			<max_angle>1.570796</max_angle>
+              		</horizontal>
+              	</scan>
+              	<range>
+              		<min>0.10</min>
+              		<max>30.0</max>
+              		<resolution>0.01</resolution>
+              	</range>
+              	<noise>
+              		<type>gaussian</type>
+              		<mean>0.0</mean>
+              		<stddev>0.01</stddev>
+              	</noise>
+            </ray>
+            <plugin name="gazebo_ros_head_ydlidar_controller" filename="libgazebo_ros_laser.so">
+            	<!-- Use topic name as /my_robot/scan -->
+				<topicName>/scan</topicName>
+				<frameName>laser_frame</frameName>
+			</plugin>
+		</sensor>
+	</gazebo>
 <!--######################################################################-->
 <gazebo>
     <plugin name="gazebo_ros_control" filename="libgazebo_ros_control.so">
-      <robotNamespace>/</robotNamespace>
       <controlPeriod>0.001</controlPeriod>
       <legacyModeNS>false</legacyModeNS>
