Commit message: Added transformations and lidar scan source file

File: urdf/rover.urdf.xacro (robot description, xacro)
@@ -14,52 +14,53 @@
     <child link="base_link"/>
   </joint>
-  <joint type="fixed" name="hokuyo_joint">
+  <!-- Add your gazebo sensors here -->
+    <gazebo reference="base_laser">
+    <sensor type="ray" name="head_hokuyo_sensor">
+      <pose>0 0 0 0 0 0</pose>
+      <visualize>false</visualize>
+      <update_rate>40</update_rate>
+      <ray>
+        <scan>
+          <horizontal>
+            <samples>720</samples>
+            <resolution>1</resolution>
+            <min_angle>-1.570796</min_angle>
+            <max_angle>1.570796</max_angle>
+          </horizontal>
+        </scan>
+        <range>
+          <min>0.8</min>
+          <max>30.0</max>
+          <resolution>0.01</resolution>
+        </range>
+        <noise>
+          <type>gaussian</type>
+          <!-- Noise parameters based on published spec for Hokuyo laser
+               achieving "+-30mm" accuracy at range < 10m.  A mean of 0.0m and
+               stddev of 0.01m will put 99.7% of samples within 0.03m of the true
+               reading. -->
+          <mean>0.0</mean>
+          <stddev>0.01</stddev>
+        </noise>
+      </ray>
+      <plugin name="gazebo_ros_head_hokuyo_controller" filename="libgazebo_ros_laser.so">
+        <topicName>/laser/scan</topicName>
+        <frameName>laser_frame</frameName>
+      </plugin>
+    </sensor>
+  </gazebo>
+<!--######################################################################-->
+<gazebo>
+    <plugin name="gazebo_ros_control" filename="libgazebo_ros_control.so">
+      <robotNamespace>/</robotNamespace>
+      <robotSimType>gazebo_ros_control/DefaultRobotHWSim</robotSimType>
+      <legacyModeNS>false</legacyModeNS>
+    </plugin>
+</gazebo>
+<joint type="fixed" name="hokuyo_joint">
     <origin xyz="0.08 0.2 0.013" rpy="0 0 0"/>
     <child link="base_laser"/>
     <parent link="base_link"/>
     <axis xyz="0 1 0" rpy="0 0 0"/>
-  </joint>
-  <gazebo reference="base_laser">
-		<gravity>true</gravity>
-		<!-- Gazebo has fixed set of Sensors types. Check them out here <> -->
-		<sensor name="laser" type="ray">
-			<!-- Add in your sensor characteristics -->
-			<pose> 0 0 0 0 0 0 </pose>
-			<visualise>true</visualise>
-			<update_rate>40</update_rate>
-			<always_on>true</always_on>
-			<ray>
-				<scan>
-					<horizontal>
-						<samples>720</samples>
-						<resolution>1</resolution>
-						<min_angle>-1.570796</min_angle>
-              			<max_angle>1.570796</max_angle>
-              		</horizontal>
-              	</scan>
-              	<range>
-              		<min>0.10</min>
-              		<max>30.0</max>
-              		<resolution>0.01</resolution>
-              	</range>
-              	<noise>
-              		<type>gaussian</type>
-              		<mean>0.0</mean>
-              		<stddev>0.01</stddev>
-              	</noise>
-            </ray>
-            <plugin name="gazebo_ros_head_ydlidar_controller" filename="libgazebo_ros_laser.so">
-            	<!-- Use topic name as /my_robot/scan -->
-				<topicName>/scan</topicName>
-				<frameName>laser_frame</frameName>
-			</plugin>
-		</sensor>
-	</gazebo>
-<!--######################################################################-->
-<gazebo>
-    <plugin name="gazebo_ros_control" filename="libgazebo_ros_control.so">
-      <controlPeriod>0.001</controlPeriod>
-      <legacyModeNS>false</legacyModeNS>
-    </plugin>
-</gazebo>
+</joint>
 </robot>

Commit message: Integrated camera and lidar. Added gripper and its controllers.

File: urdf/rover.urdf.xacro (robot description, xacro)
@@ -4,4 +4,6 @@
   <xacro:include filename="$(find rover)/urdf/Arm.urdf" />
   <xacro:include filename="$(find rover)/urdf/ydlidar.urdf" />
+  <xacro:include filename="$(find rover)/urdf/Gripper.urdf" />
+  <xacro:include filename="$(find rover)/urdf/camera.urdf" />
   <joint name="arn_base_joint" type="fixed">
     <origin rpy="0 0 0" xyz="-0.15 0.395 0.063"/>
@@ -50,4 +52,35 @@
     </sensor>
   </gazebo>
+  <gazebo reference="camera">
+    <sensor type="camera" name="camer_sensor">
+      <update_rate>30.0</update_rate>
+      <camera name="head">
+        <horizontal_fov>1.3962634</horizontal_fov>
+        <image>
+          <width>800</width>
+          <height>800</height>
+          <format>R8G8B8</format>
+        </image>
+        <clip>
+          <near>0.02</near>
+          <far>300</far>
+        </clip>
+      </camera>
+      <plugin name="camera_controller" filename="libgazebo_ros_camera.so">
+        <alwaysOn>true</alwaysOn>
+        <updateRate>0.0</updateRate>
+        <cameraName>camera</cameraName>
+        <imageTopicName>rgb/image_raw</imageTopicName>
+        <cameraInfoTopicName>rgb/camera_info</cameraInfoTopicName>
+        <frameName>camera</frameName>
+        <hackBaseline>0.07</hackBaseline>
+        <distortionK1>0.0</distortionK1>
+        <distortionK2>0.0</distortionK2>
+        <distortionK3>0.0</distortionK3>
+        <distortionT1>0.0</distortionT1>
+        <distortionT2>0.0</distortionT2>
+      </plugin>
+    </sensor>
+  </gazebo>
 <!--######################################################################-->
 <gazebo>
@@ -64,3 +97,15 @@
     <axis xyz="0 1 0" rpy="0 0 0"/>
 </joint>
+<joint type="fixed" name="gripper_joint">
+    <origin xyz="0 -0.1 -0.005" rpy="1.5708 0. 0"/>
+    <child link="gripper"/>
+    <parent link="top_wrist"/>
+    <axis xyz="1 0 0" rpy="0 0 0"/>
+</joint>
+<joint type="fixed" name="camera_joint">
+    <origin xyz="-0.15 0.30 0.11" rpy="0 0 0"/>
+    <child link="camera"/>
+    <parent link="base_link"/>
+    <axis xyz="0 1 0" rpy="0 0 0"/>
+</joint>
 </robot>
